File: PitMount.kicad_pcb (KiCad board)
At the start: 2 copper layers, 27 x 30 mm, 18 parts, among them J1 Conn_01x07, Q1 BC817, Q2 IRLML6401, U1 UnifyNano, U2 ELRS-Rx

Commit message: Fix silkscreen issues
Other:
- board text added: "+5|G|V|A|R+|R|T"
- board text removed: "+5|GND|Vid|SA|RX+|RX|TX"
Changed lines of the file:
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@@
         (effects (font (size 1.016 1.016) (thickness 0.1524)))
-    )
-    (fp_text user "+5" (at 4 -2.999999 90 unlocked) (layer "F.SilkS")
-        (effects (font (size 0.508 0.508) (thickness 0.127)))
-    )
-    (fp_text user "RX" (at 9 -2.999999 90 unlocked) (layer "F.SilkS")
-        (effects (font (size 0.508 0.508) (thickness 0.127)))
-    )
-    (fp_text user "GND" (at 1.5 -3 90 unlocked) (layer "F.SilkS")
-        (effects (font (size 0.508 0.508) (thickness 0.127)))
-    )
-    (fp_text user "TX" (at 6.5 -2.999999 90 unlocked) (layer "F.SilkS")
-        (effects (font (size 0.508 0.508) (thickness 0.127)))
     )
     (fp_text user "${REFERENCE}" (at 5.5 6.5 90 unlocked) (layer "F.Fab")
@@
     (effects (font (size 1.016 1.016) (thickness 0.1524)))
   )
-  (gr_text "+5|GND|Vid|SA|RX+|RX|TX" (at 140 100.75 270) (layer "F.SilkS")
-    (effects (font (size 0.635 0.6096) (thickness 0.1524)))
+  (gr_text "+5|G|V|A|R+|R|T" (at 139.75 100.25 270) (layer "F.SilkS")
+    (effects (font (size 1 0.9) (thickness 0.1524)))
   )
   (segment (start 160 95.5) (end 161 94.5) (width 0.635) (layer "F.Cu") (net 1))
