File: PitMount.kicad_pcb (KiCad board)
At the start: 2 copper layers, 27 x 30 mm, 18 parts, among them J1 Conn_01x07, Q1 BC817, Q2 IRLML6401, U1 UnifyNano, U2 ELRS-Rx

Commit message: Update PCB layout
Parts:
- removed H5, H6: Tooling_Hole, PitMount:Tooling Hole
- D1: footprint LED_SMD:LED_0402_1005Metric -> LED_SMD:LED_0603_1608Metric
- J1: value Conn_01x07 -> Conn_01x08_Pin
- JP1: value SolderJumper_2_Open -> Override
- TP1: value TestPoint -> PitPad
- moved J1 1.08 mm to (137.0, 94.2)
- moved D1 0.50 mm to (160.5, 105.5)
Connections:
- J1 pad 6: /RX -> GND
- J1 pad 7: /TX -> /RX
Routing:
- net /RX+5V: track 17.3 -> 20.5 mm, vias 2 -> 4
- net +5V: track 41.9 -> 40.8 mm
- net Net-(JP1-B): track 11.9 -> 12.5 mm
- net Net-(D1-A): track 1.01 -> 1.61 mm
- net Net-(D1-K): track 2.31 -> 1.80 mm
- net GND: vias 1 -> 12
Other:
- board text added: "V+ G V A R+ G R T"
- board text removed: "+5|G|V|A|R+|R|T"
